File: BEEIRON v0.0.3/BEEIRON v0.03.kicad_pcb (KiCad board)
At the start: 4 copper layers, 78 x 78 mm, 100 parts, among them J1 Conn_01x02_Male, J10 SUPPLY_OUT, J11 SUPPLY_OUT, J12 Conn_01x02_Male, J2 I2C, J3 SPI, J4 UART, J5 PWR, J6 ROTARY, J7 ISP, J8 Soldering Conn, J9 ADC, Q1 BTB26-600, SW1 SW_Push, U3 LP2985-3.3, U4 NCP1117-5.0_SOT223, U5 ATmega328P-A, U6 MAX31856, U7 MOC3020M, U8 4N25, U9 ACS712xLCTR-20A, Y1 XTY0292-7048

Commit message: added bakup file
Parts:
- removed the D3 at (169.2, 107.0)
- removed D4, D5: 1N4148W, Diode_SMD:D_SOD-123
- removed the G*** at (157.4, 102.3)
- removed the R10 at (170.2, 112.5)
- removed the R11 at (172.2, 112.5)
- removed the R12 at (174.2, 112.5)
- added JP1: Jumper_2_Open, Jumper:SolderJumper-2_P1.3mm_Open_TrianglePad1.0x1.5mm, F.Cu at (165.1, 98.0)
- added JP2: Jumper_2_Open, Jumper:SolderJumper-2_P1.3mm_Open_TrianglePad1.0x1.5mm, F.Cu at (165.1, 95.5)
- added JP3: Jumper_2_Open, Jumper:SolderJumper-2_P1.3mm_Open_TrianglePad1.0x1.5mm, F.Cu at (165.1, 93.0)
- added JP4: Jumper_2_Open, Jumper:SolderJumper-2_P1.3mm_Open_TrianglePad1.0x1.5mm, F.Cu at (165.1, 90.4)
- added JP5: Jumper_2_Open, Jumper:SolderJumper-2_P1.3mm_Open_TrianglePad1.0x1.5mm, F.Cu at (165.1, 87.9)
- added JP6: Jumper_2_Open, Jumper:SolderJumper-2_P1.3mm_Open_TrianglePad1.0x1.5mm, F.Cu at (165.1, 85.3)
- added Q1: BSS138, Package_TO_SOT_SMD:SOT-23, F.Cu at (172.3, 93.4)
- added Q2: BSS138, Package_TO_SOT_SMD:SOT-23, F.Cu at (172.3, 82.7)
- added Q3: BSS138, Package_TO_SOT_SMD:SOT-23, F.Cu at (172.3, 100.4)
- added Q4: BSS138, Package_TO_SOT_SMD:SOT-23, F.Cu at (172.3, 96.9)
- added Q5: BSS138, Package_TO_SOT_SMD:SOT-23, F.Cu at (172.3, 86.3)
- added Q6: BSS138, Package_TO_SOT_SMD:SOT-23, F.Cu at (172.3, 89.8)
- added R14: 10K, Resistor_SMD:R_0805_2012Metric, F.Cu at (175.4, 93.4)
- added R15: K10K, Resistor_SMD:R_0805_2012Metric, F.Cu at (169.3, 93.3)
- added R16: 10K, Resistor_SMD:R_0805_2012Metric, F.Cu at (175.3, 82.7)
- added R17: K10K, Resistor_SMD:R_0805_2012Metric, F.Cu at (169.3, 82.7)
- added R18: 10K, Resistor_SMD:R_0805_2012Metric, F.Cu at (175.4, 100.4)
- added R19: K10K, Resistor_SMD:R_0805_2012Metric, F.Cu at (169.3, 100.4)
- added R20: 10K, Resistor_SMD:R_0805_2012Metric, F.Cu at (175.4, 96.9)
- added R21: K10K, Resistor_SMD:R_0805_2012Metric, F.Cu at (169.3, 96.9)
- added R22: 10K, Resistor_SMD:R_0805_2012Metric, F.Cu at (175.3, 86.3)
- added R23: K10K, Resistor_SMD:R_0805_2012Metric, F.Cu at (169.3, 86.3)
- added R24: 10K, Resistor_SMD:R_0805_2012Metric, F.Cu at (175.3, 89.7)
- added R25: K10K, Resistor_SMD:R_0805_2012Metric, F.Cu at (169.3, 89.8)
- added kibuzzard-6198C887: G***, kibuzzard-6198C887, F.Cu at (161.5, 87.9)
- added kibuzzard-6198C8A0: G***, kibuzzard-6198C8A0, F.Cu at (161.5, 85.3)
- added kibuzzard-6198C8AE: G***, kibuzzard-6198C8AE, F.Cu at (161.5, 90.2)
- added kibuzzard-6198C8D5: G***, kibuzzard-6198C8D5, F.Cu at (161.9, 93.0)
- added kibuzzard-6198C8F1: G***, kibuzzard-6198C8F1, F.Cu at (161.5, 95.5)
- added kibuzzard-6198C929: G***, kibuzzard-6198C929, F.Cu at (161.0, 98.0)
- Y1: value XTY0292-7048 -> S3216000091060JY
- moved ? 43.9 mm to (133.8, 104.3)
- moved R13 16.8 mm to (177.2, 112.5), turned to 180 degrees
- moved JP7 15.1 mm to (173.6, 112.7), turned to 180 degrees
- moved J5 12.0 mm to (177.3, 109.5), turned to -90 degrees
- moved R32 10.5 mm to (166.0, 75.9)
- moved RXD1 10.5 mm to (169.4, 75.9)
- moved DL1 10.5 mm to (169.5, 71.5)
- moved DON1 10.5 mm to (169.5, 73.8)
- moved J4 10.5 mm to (175.7, 78.0)
- moved R33 10.5 mm to (166.0, 78.1)
- moved R34 10.5 mm to (166.1, 71.5)
- moved R35 10.5 mm to (166.0, 73.8)
- moved TXD1 10.5 mm to (169.4, 78.1)
- moved C15 0.33 mm to (168.1, 112.8)
- renumbered D6 to D3, JP1 to JP7, JP2 to JP8, Q1 to Q7, R13 to R10, R14 to R11, R15 to R12, R16 to R13, R17 to R26, R18 to R27, R19 to R28, R20 to R29, R21 to R30, R22 to R31, R23 to R32, R24 to R33, R25 to R34, R26 to R35, R27 to R36, R28 to R37, R29 to R38
Connections:
- BR1 pad ~: Net-(BR1-Pad~) -> (no net)
- BR2 pad ~: IRON_BLU -> (no net)
- U6 pad 10: Net-(D4-Pad2) -> SCK
- U6 pad 11: D12/SDO -> SDO
- U6 pad 12: Net-(D5-Pad2) -> SDI
- U6 pad 13: D6/FAULT -> FAULT
- U6 pad 7: D7/DDRY -> DDRY
- U6 pad 9: Net-(D3-Pad2) -> CS
Routing:
- net SDI: track 0.00 -> 48.9 mm
- net SDO: track 0.00 -> 47.2 mm, vias 0 -> 2
- net SCK: track 0.00 -> 44.4 mm, vias 0 -> 2
- net CS: track 0.00 -> 42.3 mm, vias 0 -> 2
- net DDRY: track 0.00 -> 38.4 mm, vias 0 -> 2
- net FAULT: track 0.00 -> 32.7 mm
- net D6/FAULT: track 41.7 -> 63.8 mm, vias 2 -> 4
- net Net-(D5-Pad2): track 13.0 -> 0.00 mm
- net +3V3: track 97.8 -> 110.7 mm, vias 0 -> 8
- net Net-(D4-Pad2): track 10.9 -> 0.00 mm
- net +5V: track 71.7 -> 81.8 mm, vias 57 -> 63
- net D13/SCK: track 65.2 -> 73.9 mm, vias 0 -> 2
- net Net-(D3-Pad2): track 8.02 -> 0.00 mm
- net D7/DDRY: track 30.7 -> 37.7 mm
- net D9: track 64.9 -> 58.6 mm
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Other:
- board text removed: "MAX31856"
- board text removed: "RST"
