File: BEEIRON v0.0.3/Controller.kicad_sch (KiCad schematic)
At the start: 15 parts, among them SW1 SW_Push, U5 ATmega328P-A, Y1 XTY0292-7048

Commit message: added bakup file
Parts:
- Y1: value XTY0292-7048 -> S3216000091060JY
Other:
- note added: "Cx = 2*(load cap - stray cap)-parasitic ground capacitance cx = 2(CL – CS) – CPG cx=2*(10p-3p) -4p cx=2*(7p) - 4p cx= 10p"
- note added: "ESR 10-16MHZ 100 Ω Max"
- note removed: "Cx = 2*(load cap - stray cap) cx=2*(9p-2p) cx=2*(7p) cx= 14p"
