File: BEEIRON v0.0.3/Current_Sensor.kicad_sch (KiCad schematic)
At the start: 9 parts, among them U9 ACS712xLCTR-20A

Commit message: added bakup file
Parts:
- renumbered D6 to D3, R27 to R36, R28 to R37, R29 to R38
