File: BEEIRON v0.0.4/BEEIRON v0.0.kicad_pcb (KiCad board)
At the start: 4 copper layers, 78 x 78 mm, 136 parts, among them J1 Conn_01x02_Male, J10 SUPPLY_OUT, J11 SUPPLY_OUT, J12 Conn_01x02_Male, J2 I2C, J3 SPI, J4 UART, J5 PWR, J6 ROTARY, J7 ISP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

Commit message: v0.0.4
Routing:
- net A0/CURRENT: track 60.7 -> 70.8 mm, vias 2 -> 3
- net GND: track 91.3 -> 90.6 mm, vias 31 -> 83
Other:
- rule pad_to_mask_clearance: 0.05 -> 0
- board text added: "JLCJLCJLCJLC"
